File: dwg/hBridge.sch (KiCad schematic (older format))
At the start: 17 parts

Commit message: cleaned up hbridge file
Parts:
- removed U? (x3): K847PH, symbol K847PH
- added U? (x3): K847PH, symbol K847PH
Connections:
- net labels added: FWD_HI, FWD_LO, POWER_GND, REV_HI, SIGNAL_GND
- wire segments 23 -> 34
Other:
- moved on the sheet: D?, Q?, R?

Commit message: added resistors for hbridge optocouplers
Parts:
- removed U? (x3): K847PH, symbol K847PH
- added R10, R11, R6, R7: 1k, symbol R
- added R4, R5, R8, R9: 100, symbol R
- added U3: K847PH, symbol K847PH
- gave numbers to parts that had none: 14
Connections:
- wire segments 34 -> 60
Other:
- moved on the sheet: D3, D4, D5, D6, Q1, Q2, Q5, Q6, Q7, Q8, R2, R3

Commit message: Added connectors to BOM
Parts:
- removed P11: CONN_01X03, symbol CONN_01X03
- added J16, J17, P16, P17: CONN_01X02, symbol CONN_01X02
- renumbered Q1 to Q3, Q2 to Q4, R4 to R3, R5 to R4, R6 to R5, R7 to R6, R8 to R7, R9 to R8, R3 to R9, U3 to U5, U2 to U6
Connections:
- net labels added: MTR_HI, MTR_LO
- wire segments 60 -> 46
Other:
- note added: "MOTOR"
- moved on the sheet: D3, D4, D5, D6, Q3, Q4, Q5, Q6, Q7, Q8, R10, R11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

Commit message: Added pushbuttons to layout
Parts:
- D3, D4, D5, D6: footprint (none) -> Diodes_ThroughHole:Diode_P600_Vertical_AnodeUp
- Q3, Q4, Q5, Q6, Q7, Q8: footprint (none) -> Transistors_OldSowjetAera:OldSowjetaera_Transistor_Type-II_BigPads
- R10, R11, R2, R3, R4, R5, R6, R7, R8, R9: footprint (none) -> Resistors_SMD:R_0805_HandSoldering
Changed lines of the file:
@@
 LIBS:contrib
 LIBS:valves
-LIBS:roboCooler-cache
+LIBS:roboCooler
 EELAYER 25 0
 EELAYER END
@@
 F 0 "Q7" H 6850 4750 50  0000 R CNN
 F 1 "NMOS" H 6950 4650 50  0000 R CNN
-F 2 "" H 6750 4800 29  0000 C CNN
+F 2 "Transistors_OldSowjetAera:OldSowjetaera_Transistor_Type-II_BigPads" H 6750 4800 29  0001 C CNN
 F 3 "" H 6550 4700 60  0000 C CNN
 	1    6550 4700
@@
 	4050 4900 7150 4900
 $Comp
-L GND #PWR44
+L GND #PWR040
 U 1 1 569B3E2F
 P 5600 4900
-F 0 "#PWR44" H 5600 4650 50  0001 C CNN
+F 0 "#PWR040" H 5600 4650 50  0001 C CNN
 F 1 "GND" H 5600 4750 50  0000 C CNN
 F 2 "" H 5600 4900 60  0000 C CNN
@@
 F 0 "Q6" H 6850 4350 50  0000 R CNN
 F 1 "PMOS" H 6950 4250 50  0000 R CNN
-F 2 "" H 6750 4400 29  0000 C CNN
+F 2 "Transistors_OldSowjetAera:OldSowjetaera_Transistor_Type-II_BigPads" H 6750 4400 29  0001 C CNN
 F 3 "" H 6550 4300 60  0000 C CNN
 	1    6550 4300
@@
 	4600 4100 6600 4100
 $Comp
-L +12V #PWR43
+L +12V #PWR041
 U 1 1 569B3E3D
 P 5600 4100
-F 0 "#PWR43" H 5600 3950 50  0001 C CNN
+F 0 "#PWR041" H 5600 3950 50  0001 C CNN
 F 1 "+12V" H 5600 4240 50  0000 C CNN
 F 2 "" H 5600 4100 60  0000 C CNN
@@
 F 0 "D3" H 5100 4380 50  0000 L CNN
 F 1 "D_Schottky_Small" H 4870 4220 50  0001 L CNN
-F 2 "" V 5150 4300 60  0000 C CNN
+F 2 "Diodes_ThroughHole:Diode_P600_Vertical_AnodeUp" V 5150 4300 60  0001 C CNN
 F 3 "" V 5150 4300 60  0000 C CNN
 	1    5150 4300
@@
 F 0 "D4" H 5100 4780 50  0000 L CNN
 F 1 "D_Schottky_Small" H 4870 4620 50  0001 L CNN
-F 2 "" V 5150 4700 60  0000 C CNN
+F 2 "Diodes_ThroughHole:Diode_P600_Vertical_AnodeUp" V 5150 4700 60  0001 C CNN
 F 3 "" V 5150 4700 60  0000 C CNN
 	1    5150 4700
@@
 F 0 "D6" H 6000 4780 50  0000 L CNN
 F 1 "D_Schottky_Small" H 5770 4620 50  0001 L CNN
-F 2 "" V 6050 4700 60  0000 C CNN
+F 2 "Diodes_ThroughHole:Diode_P600_Vertical_AnodeUp" V 6050 4700 60  0001 C CNN
 F 3 "" V 6050 4700 60  0000 C CNN
 	1    6050 4700
@@
 F 0 "D5" H 6000 4380 50  0000 L CNN
 F 1 "D_Schottky_Small" H 5770 4220 50  0001 L CNN
-F 2 "" V 6050 4300 60  0000 C CNN
+F 2 "Diodes_ThroughHole:Diode_P600_Vertical_AnodeUp" V 6050 4300 60  0001 C CNN
 F 3 "" V 6050 4300 60  0000 C CNN
 	1    6050 4300
@@
 F 0 "Q8" H 7550 4750 50  0000 R CNN
 F 1 "NMOS" H 7650 4650 50  0000 R CNN
-F 2 "" H 7450 4800 29  0000 C CNN
+F 2 "Transistors_OldSowjetAera:OldSowjetaera_Transistor_Type-II_BigPads" H 7450 4800 29  0001 C CNN
 F 3 "" H 7250 4700 60  0000 C CNN
 	1    7250 4700
@@
 F 0 "R9" V 6830 4100 50  0000 C CNN
 F 1 "1k" V 6750 4100 50  0000 C CNN
-F 2 "" V 6680 4100 30  0000 C CNN
+F 2 "Resistors_SMD:R_0805_HandSoldering" V 6680 4100 30  0001 C CNN
 F 3 "" H 6750 4100 30  0000 C CNN
 	1    6750 4100
@@
 F 0 "Q5" H 4950 4750 50  0000 R CNN
 F 1 "NMOS" H 5050 4650 50  0000 R CNN
-F 2 "" H 4850 4800 29  0000 C CNN
+F 2 "Transistors_OldSowjetAera:OldSowjetaera_Transistor_Type-II_BigPads" H 4850 4800 29  0001 C CNN
 F 3 "" H 4650 4700 60  0000 C CNN
 	1    4650 4700
@@
 F 0 "Q4" H 4950 4350 50  0000 R CNN
 F 1 "PMOS" H 5050 4250 50  0000 R CNN
-F 2 "" H 4850 4400 29  0000 C CNN
+F 2 "Transistors_OldSowjetAera:OldSowjetaera_Transistor_Type-II_BigPads" H 4850 4400 29  0001 C CNN
 F 3 "" H 4650 4300 60  0000 C CNN
 	1    4650 4300
@@
 F 0 "Q3" H 4250 4750 50  0000 R CNN
 F 1 "NMOS" H 4350 4650 50  0000 R CNN
-F 2 "" H 4150 4800 29  0000 C CNN
+F 2 "Transistors_OldSowjetAera:OldSowjetaera_Transistor_Type-II_BigPads" H 4150 4800 29  0001 C CNN
 F 3 "" H 3950 4700 60  0000 C CNN
 	1    3950 4700
@@
 F 0 "R2" V 4530 4100 50  0000 C CNN
 F 1 "1k" V 4450 4100 50  0000 C CNN
-F 2 "" V 4380 4100 30  0000 C CNN
+F 2 "Resistors_SMD:R_0805_HandSoldering" V 4380 4100 30  0001 C CNN
 F 3 "" H 4450 4100 30  0000 C CNN
 	1    4450 4100
@@
 POWER_GND
 $Comp
-L GND #PWR38
+L GND #PWR042
 U 1 1 569B77C8
 P 3300 1950
-F 0 "#PWR38" H 3300 1700 50  0001 C CNN
+F 0 "#PWR042" H 3300 1700 50  0001 C CNN
 F 1 "GND" H 3300 1800 50  0000 C CNN
 F 2 "" H 3300 1950 60  0000 C CNN
@@
 F 0 "U6" H 5220 3000 60  0000 C CNN
 F 1 "K847PH" H 5370 2700 60  0000 C CNN
-F 2 "" H 4750 2850 60  0000 C CNN
+F 2 "" H 4750 2850 60  0001 C CNN
 F 3 "" H 4750 2850 60  0000 C CNN
 	2    4750 2850
@@
 LID_REV_LO
 $Comp
-L GND #PWR42
+L GND #PWR043
 U 1 1 569B8D1F
 P 5000 3400
-F 0 "#PWR42" H 5000 3150 50  0001 C CNN
+F 0 "#PWR043" H 5000 3150 50  0001 C CNN
 F 1 "GND" H 5000 3250 50  0000 C CNN
 F 2 "" H 5000 3400 60  0000 C CNN
@@
 F 0 "R4" V 4680 2450 50  0000 C CNN
 F 1 "100" V 4600 2450 50  0000 C CNN
-F 2 "" V 4530 2450 30  0000 C CNN
+F 2 "Resistors_SMD:R_0805_HandSoldering" V 4530 2450 30  0001 C CNN
 F 3 "" H 4600 2450 30  0000 C CNN
 	1    4600 2450
@@
 F 0 "R6" V 5080 3250 50  0000 C CNN
 F 1 "1k" V 5000 3250 50  0000 C CNN
-F 2 "" V 4930 3250 30  0000 C CNN
+F 2 "Resistors_SMD:R_0805_HandSoldering" V 4930 3250 30  0001 C CNN
 F 3 "" H 5000 3250 30  0000 C CNN
 	1    5000 3250
@@
 $EndComp
 $Comp
-L +12V #PWR41
+L +12V #PWR044
 U 1 1 569A6C93
 P 5000 2650
-F 0 "#PWR41" H 5000 2500 50  0001 C CNN
+F 0 "#PWR044" H 5000 2500 50  0001 C CNN
 F 1 "+12V" H 5000 2790 50  0000 C CNN
 F 2 "" H 5000 2650 60  0000 C CNN
@@
 F 0 "U5" H 7020 3000 60  0000 C CNN
 F 1 "K847PH" H 7170 2700 60  0000 C CNN
-F 2 "" H 6550 2850 60  0000 C CNN
+F 2 "" H 6550 2850 60  0001 C CNN
 F 3 "" H 6550 2850 60  0000 C CNN
 	3    6550 2850
@@
 $EndComp
 $Comp
-L GND #PWR48
+L GND #PWR045
 U 1 1 569AAB67
 P 6800 3400
-F 0 "#PWR48" H 6800 3150 50  0001 C CNN
+F 0 "#PWR045" H 6800 3150 50  0001 C CNN
 F 1 "GND" H 6800 3250 50  0000 C CNN
 F 2 "" H 6800 3400 60  0000 C CNN
@@
 F 0 "R8" V 6480 2450 50  0000 C CNN
 F 1 "100" V 6400 2450 50  0000 C CNN
-F 2 "" V 6330 2450 30  0000 C CNN
+F 2 "Resistors_SMD:R_0805_HandSoldering" V 6330 2450 30  0001 C CNN
 F 3 "" H 6400 2450 30  0000 C CNN
 	1    6400 2450
@@
 F 0 "R11" V 6880 3250 50  0000 C CNN
 F 1 "1k" V 6800 3250 50  0000 C CNN
-F 2 "" V 6730 3250 30  0000 C CNN
+F 2 "Resistors_SMD:R_0805_HandSoldering" V 6730 3250 30  0001 C CNN
 F 3 "" H 6800 3250 30  0000 C CNN
 	1    6800 3250
@@
 $EndComp
 $Comp
-L +12V #PWR47
+L +12V #PWR046
 U 1 1 569AAB7E
 P 6800 2650
-F 0 "#PWR47" H 6800 2500 50  0001 C CNN
+F 0 "#PWR046" H 6800 2500 50  0001 C CNN
 F 1 "+12V" H 6800 2790 50  0000 C CNN
 F 2 "" H 6800 2650 60  0000 C CNN
@@
 F 0 "U5" H 5220 1550 60  0000 C CNN
 F 1 "K847PH" H 5370 1250 60  0000 C CNN
-F 2 "" H 4750 1400 60  0000 C CNN
+F 2 "" H 4750 1400 60  0001 C CNN
 F 3 "" H 4750 1400 60  0000 C CNN
 	1    4750 1400
@@
 $EndComp
 $Comp
-L GND #PWR40
+L GND #PWR047
 U 1 1 569AAE5C
 P 5000 1950
-F 0 "#PWR40" H 5000 1700 50  0001 C CNN
+F 0 "#PWR047" H 5000 1700 50  0001 C CNN
 F 1 "GND" H 5000 1800 50  0000 C CNN
 F 2 "" H 5000 1950 60  0000 C CNN
@@
 F 0 "R3" V 4680 1000 50  0000 C CNN
 F 1 "100" V 4600 1000 50  0000 C CNN
-F 2 "" V 4530 1000 30  0000 C CNN
+F 2 "Resistors_SMD:R_0805_HandSoldering" V 4530 1000 30  0001 C CNN
 F 3 "" H 4600 1000 30  0000 C CNN
 	1    4600 1000
@@
 F 0 "R5" V 5080 1800 50  0000 C CNN
 F 1 "1k" V 5000 1800 50  0000 C CNN
-F 2 "" V 4930 1800 30  0000 C CNN
+F 2 "Resistors_SMD:R_0805_HandSoldering" V 4930 1800 30  0001 C CNN
 F 3 "" H 5000 1800 30  0000 C CNN
 	1    5000 1800
@@
 $EndComp
 $Comp
-L +12V #PWR39
+L +12V #PWR048
 U 1 1 569AAE73
 P 5000 1200
-F 0 "#PWR39" H 5000 1050 50  0001 C CNN
+F 0 "#PWR048" H 5000 1050 50  0001 C CNN
 F 1 "+12V" H 5000 1340 50  0000 C CNN
 F 2 "" H 5000 1200 60  0000 C CNN
@@
 F 0 "U5" H 7020 1550 60  0000 C CNN
 F 1 "K847PH" H 7170 1250 60  0000 C CNN
-F 2 "" H 6550 1400 60  0000 C CNN
+F 2 "" H 6550 1400 60  0001 C CNN
 F 3 "" H 6550 1400 60  0000 C CNN
 	2    6550 1400
@@
 $EndComp
 $Comp
-L GND #PWR46
+L GND #PWR049
 U 1 1 569AAE83
 P 6800 1950
-F 0 "#PWR46" H 6800 1700 50  0001 C CNN
+F 0 "#PWR049" H 6800 1700 50  0001 C CNN
 F 1 "GND" H 6800 1800 50  0000 C CNN
 F 2 "" H 6800 1950 60  0000 C CNN
@@
 F 0 "R7" V 6480 1000 50  0000 C CNN
 F 1 "100" V 6400 1000 50  0000 C CNN
-F 2 "" V 6330 1000 30  0000 C CNN
+F 2 "Resistors_SMD:R_0805_HandSoldering" V 6330 1000 30  0001 C CNN
 F 3 "" H 6400 1000 30  0000 C CNN
 	1    6400 1000
@@
 F 0 "R10" V 6880 1800 50  0000 C CNN
 F 1 "1k" V 6800 1800 50  0000 C CNN
-F 2 "" V 6730 1800 30  0000 C CNN
+F 2 "Resistors_SMD:R_0805_HandSoldering" V 6730 1800 30  0001 C CNN
 F 3 "" H 6800 1800 30  0000 C CNN
 	1    6800 1800
@@
 $EndComp
 $Comp
-L +12V #PWR45
+L +12V #PWR050
 U 1 1 569AAE9A
 P 6800 1200
-F 0 "#PWR45" H 6800 1050 50  0001 C CNN
+F 0 "#PWR050" H 6800 1050 50  0001 C CNN
 F 1 "+12V" H 6800 1340 50  0000 C CNN
 F 2 "" H 6800 1200 60  0000 C CNN
@@
 F 0 "J16" H 4350 5950 50  0000 C CNN
 F 1 "CONN_01X02" V 4450 5800 50  0000 C CNN
-F 2 "" H 4350 5800 60  0000 C CNN
+F 2 "" H 4350 5800 60  0001 C CNN
 F 3 "" H 4350 5800 60  0000 C CNN
 	1    4350 5800
@@
 F 0 "P16" H 4700 5950 50  0000 C CNN
 F 1 "CONN_01X02" V 4800 5800 50  0000 C CNN
-F 2 "" H 4700 5800 60  0000 C CNN
+F 2 "" H 4700 5800 60  0001 C CNN
 F 3 "" H 4700 5800 60  0000 C CNN
 	1    4700 5800
@@
 F 0 "J17" H 6700 5950 50  0000 C CNN
 F 1 "CONN_01X02" V 6800 5800 50  0000 C CNN
-F 2 "" H 6700 5800 60  0000 C CNN
+F 2 "" H 6700 5800 60  0001 C CNN
 F 3 "" H 6700 5800 60  0000 C CNN
 	1    6700 5800
@@
 F 0 "P17" H 6350 5950 50  0000 C CNN
 F 1 "CONN_01X02" V 6450 5800 50  0000 C CNN
-F 2 "" H 6350 5800 60  0000 C CNN
+F 2 "" H 6350 5800 60  0001 C CNN
 F 3 "" H 6350 5800 60  0000 C CNN
 	1    6350 5800
