File: dwg/roboCooler.sch (KiCad schematic (older format))
At the start: 37 parts, among them J1 CONN_02X25, J10 CONN_01X12, J11 CONN_01X12, J12 CONN_01X04, J13 CONN_01X04, J14 CONN_01X04, J15 CONN_01X04, J2 CONN_02X25, J3 CONN_01X04, J4 CONN_01X04, J5 CONN_01X02, J6 CONN_01X02, J7 CONN_01X02, J8 CONN_01X02, J9 CONN_01X06, P13 CONN_01X04, P15 CONN_01X04, P3 CONN_01X04, P4 CONN_01X04, P5 CONN_01X02, P6 CONN_01X02, P7 CONN_01X02, P8 CONN_01X02, Q1 NMOS, Q2 NMOS, SW1 SPST_4PIN, SW2 SPST_4PIN, U2 4069, U3 HALL_EFFECT, U4 HALL_EFFECT

Commit message: Added LED USART to layout
Parts:
- removed J4, P3, P4: CONN_01X04, symbol CONN_01X04
- removed U2: 4069, symbol 4069
- added C1: .01UF, Capacitors_SMD:C_0805_HandSoldering, symbol C
- added C2: 1UF, Capacitors_SMD:C_0805_HandSoldering, symbol C
- added U1: SN74LV, TO_SOT_Packages_SMD:SOT-23-5, symbol 74AHC1G14
Connections:
- no-connect marks 16 -> 18
Other:
- moved on the sheet: J3, R1
Changed lines of the file:
@@
-$EndComp
-$Comp
-L 4069 U2
-U 1 1 5665387C
-P 6900 1400
-F 0 "U2" H 7095 1515 60  0000 C CNN
-F 1 "4069" H 7090 1275 60  0001 C CNN
-F 2 "" H 6900 1400 60  0001 C CNN
-F 3 "" H 6900 1400 60  0000 C CNN
-	1    6900 1400
-	1    0    0    -1
 $EndComp
 $Comp
 L R R1
 U 1 1 56653A46
-P 7350 1250
-F 0 "R1" V 7430 1250 50  0000 C CNN
-F 1 "1k" V 7350 1250 50  0000 C CNN
-F 2 "Resistors_SMD:R_0805_HandSoldering" V 7280 1250 30  0001 C CNN
-F 3 "" H 7350 1250 30  0000 C CNN
-	1    7350 1250
+P 6075 1225
+F 0 "R1" V 6155 1225 50  0000 C CNN
+F 1 "1k" V 6075 1225 50  0000 C CNN
+F 2 "Resistors_SMD:R_0805_HandSoldering" V 6005 1225 30  0001 C CNN
+F 3 "" H 6075 1225 30  0000 C CNN
+	1    6075 1225
 	1    0    0    -1
 $EndComp
@@
 L +5V #PWR05
 U 1 1 56653B39
-P 7350 1100
-F 0 "#PWR05" H 7350 950 50  0001 C CNN
-F 1 "+5V" H 7350 1240 50  0000 C CNN
-F 2 "" H 7350 1100 60  0000 C CNN
-F 3 "" H 7350 1100 60  0000 C CNN
-	1    7350 1100
+P 6075 1075
+F 0 "#PWR05" H 6075 925 50  0001 C CNN
+F 1 "+5V" H 6075 1215 50  0000 C CNN
+F 2 "" H 6075 1075 60  0000 C CNN
+F 3 "" H 6075 1075 60  0000 C CNN
+	1    6075 1075
 	1    0    0    -1
 $EndComp
@@
 L GND #PWR06
 U 1 1 56653BAF
-P 7800 1600
-F 0 "#PWR06" H 7800 1350 50  0001 C CNN
-F 1 "GND" H 7800 1450 50  0000 C CNN
-F 2 "" H 7800 1600 60  0000 C CNN
-F 3 "" H 7800 1600 60  0000 C CNN
-	1    7800 1600
+P 6525 1575
+F 0 "#PWR06" H 6525 1325 50  0001 C CNN
+F 1 "GND" H 6525 1425 50  0000 C CNN
+F 2 "" H 6525 1575 60  0000 C CNN
+F 3 "" H 6525 1575 60  0000 C CNN
+	1    6525 1575
 	1    0    0    -1
 $EndComp
@@
 L +5V #PWR07
 U 1 1 56653C03
-P 7800 1300
-F 0 "#PWR07" H 7800 1150 50  0001 C CNN
-F 1 "+5V" H 7800 1440 50  0000 C CNN
-F 2 "" H 7800 1300 60  0000 C CNN
-F 3 "" H 7800 1300 60  0000 C CNN
-	1    7800 1300
+P 6525 1275
+F 0 "#PWR07" H 6525 1125 50  0001 C CNN
+F 1 "+5V" H 6525 1415 50  0000 C CNN
+F 2 "" H 6525 1275 60  0000 C CNN
+F 3 "" H 6525 1275 60  0000 C CNN
+	1    6525 1275
 	1    0    0    -1
 $EndComp
@@
 	1    0    0    -1
 $EndComp
-Text GLabel 3150 1800 0    60   Input ~ 0
+Text GLabel 1700 1400 2    60   Input ~ 0
 LED_UART
-Text GLabel 6450 1400 0    60   Input ~ 0
+Text GLabel 5175 1375 0    60   Input ~ 0
 LED_UART
 Text GLabel 3150 1700 0    60   Input ~ 0
@@
 L CONN_01X04 J3
 U 1 1 569C5091
-P 8000 1450
-F 0 "J3" H 8000 1700 50  0000 C CNN
-F 1 "CONN_01X04" V 8100 1450 50  0000 C CNN
-F 2 "Socket_Strips:Socket_Strip_Angled_1x04" H 8000 1450 60  0001 C CNN
-F 3 "" H 8000 1450 60  0000 C CNN
-	1    8000 1450
+P 6725 1425
+F 0 "J3" H 6725 1675 50  0000 C CNN
+F 1 "CONN_01X04" V 6825 1425 50  0000 C CNN
+F 2 "Socket_Strips:Socket_Strip_Angled_1x04" H 6725 1425 60  0001 C CNN
+F 3 "" H 6725 1425 60  0000 C CNN
+	1    6725 1425
 	1    0    0    -1
 $EndComp
@@
 	1    0    0    -1
 $EndComp
-$Comp
-L CONN_01X04 P3
-U 1 1 569D054B
-P 8350 1450
-F 0 "P3" H 8350 1700 50  0000 C CNN
-F 1 "CONN_01X04" V 8450 1450 50  0000 C CNN
-F 2 "" H 8350 1450 60  0001 C CNN
-F 3 "" H 8350 1450 60  0000 C CNN
-	1    8350 1450
-	-1   0    0    -1
-$EndComp
-$Comp
-L CONN_01X04 J4
-U 1 1 569D1795
-P 10350 1450
-F 0 "J4" H 10350 1700 50  0000 C CNN
-F 1 "CONN_01X04" V 10450 1450 50  0000 C CNN
-F 2 "" H 10350 1450 60  0001 C CNN
-F 3 "" H 10350 1450 60  0000 C CNN
-	1    10350 1450
-	-1   0    0    -1
-$EndComp
-$Comp
-L CONN_01X04 P4
-U 1 1 569D179B
-P 10000 1450
-F 0 "P4" H 10000 1700 50  0000 C CNN
-F 1 "CONN_01X04" V 10100 1450 50  0000 C CNN
-F 2 "" H 10000 1450 60  0001 C CNN
-F 3 "" H 10000 1450 60  0000 C CNN
-	1    10000 1450
-	1    0    0    -1
-$EndComp
-Text Notes 10650 1450 0    60   ~ 0
+Text Notes 6925 1425 0    60   ~ 0
 LED STRIP
 $Comp
@@
 Connection ~ 7800 2400
 Wire Wire Line
-	7350 1400 7800 1400
+	6075 1375 6525 1375
 Wire Wire Line
 	7300 5350 9800 5350
@@
 Wire Wire Line
 	7800 3400 7800 3450
-Wire Notes Line
-	8600 1450 9750 1450
 Wire Notes Line
 	8600 2300 9750 2300
@@
 NoConn ~ 3150 1600
 NoConn ~ 3150 1200
+$Comp
+L GND #PWR042
+U 1 1 5767C7E8
+P 5575 1575
+F 0 "#PWR042" H 5575 1325 50  0001 C CNN
+F 1 "GND" H 5575 1425 50  0000 C CNN
+F 2 "" H 5575 1575 60  0000 C CNN
+F 3 "" H 5575 1575 60  0000 C CNN
+	1    5575 1575
+	1    0    0    -1
+$EndComp
+$Comp
+L +5V #PWR043
+U 1 1 5767C8A6
+P 5575 1175
+F 0 "#PWR043" H 5575 1025 50  0001 C CNN
+F 1 "+5V" H 5575 1315 50  0000 C CNN
+F 2 "" H 5575 1175 60  0000 C CNN
+F 3 "" H 5575 1175 60  0000 C CNN
+	1    5575 1175
+	1    0    0    -1
+$EndComp
+$Comp
+L 74AHC1G14 U1
+U 1 1 5767C49F
+P 5625 1375
+F 0 "U1" H 5770 1490 50  0000 C CNN
+F 1 "SN74LV" H 5825 1275 50  0001 C CNN
+F 2 "TO_SOT_Packages_SMD:SOT-23-5" H 5720 1240 50  0001 C CNN
+F 3 "" H 5770 1490 50  0000 C CNN
+	1    5625 1375
+	1    0    0    -1
+$EndComp
+NoConn ~ 6525 1475
+NoConn ~ 3150 2200
+$Comp
+L C C1
+U 1 1 57681FCF
+P 7625 1375
+F 0 "C1" H 7650 1475 50  0000 L CNN
+F 1 ".01UF" H 7650 1275 50  0000 L CNN
+F 2 "Capacitors_SMD:C_0805_HandSoldering" H 7663 1225 50  0001 C CNN
+F 3 "" H 7625 1375 50  0000 C CNN
+	1    7625 1375
+	1    0    0    -1
+$EndComp
+$Comp
+L +5V #PWR044
+U 1 1 57682EDC
+P 7625 1225
+F 0 "#PWR044" H 7625 1075 50  0001 C CNN
+F 1 "+5V" H 7625 1365 50  0000 C CNN
+F 2 "" H 7625 1225 60  0000 C CNN
+F 3 "" H 7625 1225 60  0000 C CNN
+	1    7625 1225
+	1    0    0    -1
+$EndComp
+$Comp
+L GND #PWR045
+U 1 1 57682F8C
+P 7625 1525
+F 0 "#PWR045" H 7625 1275 50  0001 C CNN
+F 1 "GND" H 7625 1375 50  0000 C CNN
+F 2 "" H 7625 1525 60  0000 C CNN
+F 3 "" H 7625 1525 60  0000 C CNN
+	1    7625 1525
+	1    0    0    -1
+$EndComp
+$Comp
+L C C2
+U 1 1 57683D72
+P 7900 1375
+F 0 "C2" H 7925 1475 50  0000 L CNN
+F 1 "1UF" H 7925 1275 50  0000 L CNN
+F 2 "Capacitors_SMD:C_0805_HandSoldering" H 7938 1225 50  0001 C CNN
+F 3 "" H 7900 1375 50  0000 C CNN
+	1    7900 1375
+	1    0    0    -1
+$EndComp
+$Comp
+L +5V #PWR046
+U 1 1 57683D78
+P 7900 1225
+F 0 "#PWR046" H 7900 1075 50  0001 C CNN
+F 1 "+5V" H 7900 1365 50  0000 C CNN
+F 2 "" H 7900 1225 60  0000 C CNN
+F 3 "" H 7900 1225 60  0000 C CNN
+	1    7900 1225
+	1    0    0    -1
+$EndComp
+$Comp
+L GND #PWR047
+U 1 1 57683D7E
+P 7900 1525
+F 0 "#PWR047" H 7900 1275 50  0001 C CNN
+F 1 "GND" H 7900 1375 50  0000 C CNN
+F 2 "" H 7900 1525 60  0000 C CNN
+F 3 "" H 7900 1525 60  0000 C CNN
+	1    7900 1525
+	1    0    0    -1
+$EndComp
 $EndSCHEMATC

Commit message: added fan driver components to layout
Parts:
- removed J6, P5, P6: CONN_01X02, symbol CONN_01X02
- added C3: .01UF, Capacitors_SMD:C_0805_HandSoldering, symbol C
- added C4: 1UF, Capacitors_SMD:C_0805_HandSoldering, symbol C
- C1: footprint Capacitors_SMD:C_0805_HandSoldering -> TO_SOT_Packages_SMD:TO-263-3Lead
- D1: value D_Schottky_Small -> BAT42; footprint Diodes_ThroughHole:Diode_P600_Vertical_AnodeUp -> Diodes_SMD:SOD-123
- Q1: footprint Transistors_OldSowjetAera:OldSowjetaera_Transistor_Type-II_BigPads -> TO_SOT_Packages_SMD:TO-252-2Lead
Other:
- moved on the sheet: D1, J5, Q1
Changed lines of the file:
@@
 L D_Schottky_Small D1
 U 1 1 566526F5
-P 7650 2300
-F 0 "D1" H 7600 2380 50  0000 L CNN
-F 1 "D_Schottky_Small" H 7370 2220 50  0001 L CNN
-F 2 "Diodes_ThroughHole:Diode_P600_Vertical_AnodeUp" V 7650 2300 60  0001 C CNN
-F 3 "" V 7650 2300 60  0000 C CNN
-	1    7650 2300
+P 5425 2250
+F 0 "D1" H 5375 2330 50  0000 L CNN
+F 1 "BAT42" H 5145 2170 50  0001 L CNN
+F 2 "Diodes_SMD:SOD-123" V 5425 2250 60  0001 C CNN
+F 3 "http://www.digikey.com/product-search/en/discrete-semiconductor-products/diodes-rectifiers-single/1376383?k=BAT42W-TP&k=&pkeyword=BAT42W-TP&pv7=2&mnonly=0&newproducts=0&ColumnSort=0&page=1&quantity=0&ptm=0&fid=0&pageSize=25" H 5425 2250 60  0001 C CNN
+	1    5425 2250
 	0    -1   1    0
 $EndComp
@@
 L +12V #PWR03
 U 1 1 56652701
-P 7800 2200
-F 0 "#PWR03" H 7800 2050 50  0001 C CNN
-F 1 "+12V" H 7800 2340 50  0000 C CNN
-F 2 "" H 7800 2200 60  0000 C CNN
-F 3 "" H 7800 2200 60  0000 C CNN
-	1    7800 2200
+P 5575 2150
+F 0 "#PWR03" H 5575 2000 50  0001 C CNN
+F 1 "+12V" H 5575 2290 50  0000 C CNN
+F 2 "" H 5575 2150 60  0000 C CNN
+F 3 "" H 5575 2150 60  0000 C CNN
+	1    5575 2150
 	1    0    0    -1
 $EndComp
@@
 L Q_NMOS_DGS Q1
 U 1 1 56652707
-P 7700 2650
-F 0 "Q1" H 8000 2700 50  0000 R CNN
-F 1 "NMOS" H 8100 2600 50  0000 R CNN
-F 2 "Transistors_OldSowjetAera:OldSowjetaera_Transistor_Type-II_BigPads" H 7900 2750 29  0001 C CNN
-F 3 "" H 7700 2650 60  0000 C CNN
-	1    7700 2650
+P 5475 2600
+F 0 "Q1" H 5775 2650 50  0000 R CNN
+F 1 "NMOS" H 5875 2550 50  0000 R CNN
+F 2 "TO_SOT_Packages_SMD:TO-252-2Lead" H 5675 2700 29  0001 C CNN
+F 3 "" H 5475 2600 60  0000 C CNN
+	1    5475 2600
 	1    0    0    -1
 $EndComp
@@
 L GND #PWR04
 U 1 1 56652712
-P 7800 2850
-F 0 "#PWR04" H 7800 2600 50  0001 C CNN
-F 1 "GND" H 7800 2700 50  0000 C CNN
-F 2 "" H 7800 2850 60  0000 C CNN
-F 3 "" H 7800 2850 60  0000 C CNN
-	1    7800 2850
+P 5575 2800
+F 0 "#PWR04" H 5575 2550 50  0001 C CNN
+F 1 "GND" H 5575 2650 50  0000 C CNN
+F 2 "" H 5575 2800 60  0000 C CNN
+F 3 "" H 5575 2800 60  0000 C CNN
+	1    5575 2800
 	1    0    0    -1
 $EndComp
@@
 Text GLabel 7500 3850 0    60   Input ~ 0
 PUMP
-Text GLabel 1950 1600 2    60   Input ~ 0
+Text GLabel 1200 1300 0    60   Input ~ 0
 FAN
-Text GLabel 7500 2650 0    60   Input ~ 0
+Text GLabel 5275 2600 0    60   Input ~ 0
 FAN
 Text GLabel 950  5350 0    60   Input ~ 0
@@
 L CONN_01X02 J5
 U 1 1 569C0367
-P 8000 2300
-F 0 "J5" H 8000 2450 50  0000 C CNN
-F 1 "CONN_01X02" V 8100 2300 50  0000 C CNN
-F 2 "Socket_Strips:Socket_Strip_Angled_1x02" H 8000 2300 60  0001 C CNN
-F 3 "" H 8000 2300 60  0000 C CNN
-	1    8000 2300
+P 5775 2250
+F 0 "J5" H 5775 2400 50  0000 C CNN
+F 1 "CONN_01X02" V 5875 2250 50  0000 C CNN
+F 2 "Socket_Strips:Socket_Strip_Angled_1x02" H 5775 2250 60  0001 C CNN
+F 3 "" H 5775 2250 60  0000 C CNN
+	1    5775 2250
 	1    0    0    -1
 $EndComp
@@
 Text Notes 6925 1425 0    60   ~ 0
 LED STRIP
-$Comp
-L CONN_01X02 P5
-U 1 1 569D4F19
-P 8350 2300
-F 0 "P5" H 8350 2450 50  0000 C CNN
-F 1 "CONN_01X02" V 8450 2300 50  0000 C CNN
-F 2 "" H 8350 2300 60  0001 C CNN
-F 3 "" H 8350 2300 60  0000 C CNN
-	1    8350 2300
-	-1   0    0    -1
-$EndComp
-$Comp
-L CONN_01X02 J6
-U 1 1 569D5945
-P 10350 2300
-F 0 "J6" H 10350 2450 50  0000 C CNN
-F 1 "CONN_01X02" V 10450 2300 50  0000 C CNN
-F 2 "" H 10350 2300 60  0001 C CNN
-F 3 "" H 10350 2300 60  0000 C CNN
-	1    10350 2300
-	-1   0    0    -1
-$EndComp
-$Comp
-L CONN_01X02 P6
-U 1 1 569D594B
-P 10000 2300
-F 0 "P6" H 10000 2450 50  0000 C CNN
-F 1 "CONN_01X02" V 10100 2300 50  0000 C CNN
-F 2 "" H 10000 2300 60  0001 C CNN
-F 3 "" H 10000 2300 60  0000 C CNN
-	1    10000 2300
-	1    0    0    -1
-$EndComp
-Text Notes 10650 2350 0    60   ~ 0
+Text Notes 6025 2300 0    60   ~ 0
 FAN
 $Comp
@@
 Connection ~ 7800 3600
 Wire Wire Line
-	7800 2350 7800 2450
-Wire Wire Line
-	7650 2200 7800 2200
-Wire Wire Line
-	7800 2400 7650 2400
-Connection ~ 7800 2400
+	5575 2300 5575 2400
+Wire Wire Line
+	5425 2150 5575 2150
+Wire Wire Line
+	5575 2350 5425 2350
+Connection ~ 5575 2350
 Wire Wire Line
 	6075 1375 6525 1375
@@
 	7300 4700 9800 4700
 Wire Wire Line
-	7800 2200 7800 2250
+	5575 2150 5575 2200
 Wire Wire Line
 	7800 3400 7800 3450
-Wire Notes Line
-	8600 2300 9750 2300
 Wire Notes Line
 	8600 3500 9750 3500
@@
 F 0 "C1" H 7650 1475 50  0000 L CNN
 F 1 ".01UF" H 7650 1275 50  0000 L CNN
-F 2 "Capacitors_SMD:C_0805_HandSoldering" H 7663 1225 50  0001 C CNN
+F 2 "TO_SOT_Packages_SMD:TO-263-3Lead" H 7663 1225 50  0001 C CNN
 F 3 "" H 7625 1375 50  0000 C CNN
 	1    7625 1375
@@
 	1    0    0    -1
 $EndComp
+$Comp
+L C C3
+U 1 1 576882DB
+P 7625 2275
+F 0 "C3" H 7650 2375 50  0000 L CNN
+F 1 ".01UF" H 7650 2175 50  0000 L CNN
+F 2 "Capacitors_SMD:C_0805_HandSoldering" H 7663 2125 50  0001 C CNN
+F 3 "" H 7625 2275 50  0000 C CNN
+	1    7625 2275
+	1    0    0    -1
+$EndComp
+$Comp
+L GND #PWR049
+U 1 1 576882E7
+P 7625 2425
+F 0 "#PWR049" H 7625 2175 50  0001 C CNN
+F 1 "GND" H 7625 2275 50  0000 C CNN
+F 2 "" H 7625 2425 60  0000 C CNN
+F 3 "" H 7625 2425 60  0000 C CNN
+	1    7625 2425
+	1    0    0    -1
+$EndComp
+$Comp
+L C C4
+U 1 1 576882ED
+P 7900 2275
+F 0 "C4" H 7925 2375 50  0000 L CNN
+F 1 "1UF" H 7925 2175 50  0000 L CNN
+F 2 "Capacitors_SMD:C_0805_HandSoldering" H 7938 2125 50  0001 C CNN
+F 3 "" H 7900 2275 50  0000 C CNN
+	1    7900 2275
+	1    0    0    -1
+$EndComp
+$Comp
+L GND #PWR051
+U 1 1 576882F9
+P 7900 2425
+F 0 "#PWR051" H 7900 2175 50  0001 C CNN
+F 1 "GND" H 7900 2275 50  0000 C CNN
+F 2 "" H 7900 2425 60  0000 C CNN
+F 3 "" H 7900 2425 60  0000 C CNN
+	1    7900 2425
+	1    0    0    -1
+$EndComp
+$Comp
+L +12V #PWR?
+U 1 1 576BE39C
+P 7625 2125
+F 0 "#PWR?" H 7625 1975 50  0001 C CNN
+F 1 "+12V" H 7625 2265 50  0000 C CNN
+F 2 "" H 7625 2125 60  0000 C CNN
+F 3 "" H 7625 2125 60  0000 C CNN
+	1    7625 2125
+	1    0    0    -1
+$EndComp
+$Comp
+L +12V #PWR?
+U 1 1 576BE44C
+P 7900 2125
+F 0 "#PWR?" H 7900 1975 50  0001 C CNN
+F 1 "+12V" H 7900 2265 50  0000 C CNN
+F 2 "" H 7900 2125 60  0000 C CNN
+F 3 "" H 7900 2125 60  0000 C CNN
+	1    7900 2125
+	1    0    0    -1
+$EndComp

Commit message: added pump parts to layout
Parts:
- removed J7: CONN_01X02, Socket_Strips:Socket_Strip_Angled_1x02, symbol CONN_01X02
- removed J8, P7, P8: CONN_01X02, symbol CONN_01X02
- added C5: .01UF, Capacitors_SMD:C_0805_HandSoldering, symbol C
- added C6: 1UF, Capacitors_SMD:C_0805_HandSoldering, symbol C
- added J4: CONN_01X02, Socket_Strips:Socket_Strip_Angled_1x02, symbol CONN_01X02
- D2: value D_Schottky_Small -> BAT42; footprint Diodes_ThroughHole:Diode_P600_Vertical_AnodeUp -> Diodes_SMD:SOD-123
- J9: footprint Pin_Headers:Pin_Header_Straight_1x06 -> Socket_Strips:Socket_Strip_Straight_1x06
- Q2: footprint Transistors_OldSowjetAera:OldSowjetaera_Transistor_Type-II_BigPads -> TO_SOT_Packages_SMD:TO-252-2Lead

Commit message: added hall sensors to layout
Parts:
- removed U3, U4: HALL_EFFECT, symbol HALL_EFFECT
- added C7, C8: .1UF, Capacitors_SMD:C_0805_HandSoldering, symbol C
- added P1, P2: CONN_01X03, Socket_Strips:Socket_Strip_Angled_1x03, symbol CONN_01X03
Connections:
- wire segments 33 -> 27
